File: EMC.kicad_pcb (KiCad board)
At the start: 2 copper layers, 57 x 159 mm, 27 parts, among them J1 PWR, J2 TEMP, J3 HALL, J4 IN, J5 OUT, J6 MPWR, J7 MCTL, Q1 Q_PMOS_GDS

Commit message: Small fixes
Connections:
- J5 pad 6: +12V -> VCC
Routing:
- net VCC: track 35.4 -> 63.3 mm
- net +12V: track 148.6 -> 138.0 mm
- added copper zone on B.Cu, net GND
Changed lines of the file:
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@@
   )
   (setup
-    (last_trace_width 0.25)
+    (last_trace_width 2)
     (user_trace_width 0.5)
     (user_trace_width 1)
@@
       (net 7 GND))
     (pad 6 thru_hole circle (at 25.4 0 90) (size 3 3) (drill 1.52) (layers *.Cu *.Mask)
-      (net 27 +12V))
+      (net 30 VCC))
     (model ${KISYS3DMOD}/TerminalBlock.3dshapes/TerminalBlock_bornier-6_P5.08mm.wrl
       (offset (xyz 12.69999980926514 0 0))
@@
   (segment (start 189.3 82.15) (end 195.85 82.15) (width 2) (layer F.Cu) (net 27))
   (segment (start 196 82) (end 202 82) (width 2) (layer F.Cu) (net 27))
-  (segment (start 213 80.6) (end 211.6 82) (width 2) (layer B.Cu) (net 27))
-  (segment (start 211.6 82) (end 209.5 82) (width 2) (layer B.Cu) (net 27))
   (segment (start 201.5 132.5) (end 196.5 132.5) (width 2) (layer B.Cu) (net 27))
   (segment (start 209.5 108.066798) (end 211.5 110.066798) (width 2) (layer B.Cu) (net 27))
@@
   (segment (start 207.5 82) (end 209.5 84) (width 2) (layer B.Cu) (net 27))
   (segment (start 205 82) (end 207.5 82) (width 2) (layer B.Cu) (net 27))
-  (segment (start 209.5 82) (end 205 82) (width 2) (layer B.Cu) (net 27))
   (segment (start 205 82) (end 202 82) (width 2) (layer B.Cu) (net 27))
-  (segment (start 209.5 82) (end 209.5 84) (width 2) (layer B.Cu) (net 27))
   (segment (start 209.5 84) (end 209.5 108.066798) (width 2) (layer B.Cu) (net 27))
   (segment (start 211 112.5) (end 211.5 112) (width 0.5) (layer B.Cu) (net 27))
@@
   (segment (start 187 84.5) (end 186 85.5) (width 2) (layer F.Cu) (net 30))
   (segment (start 187 75.85) (end 187 82.15) (width 2) (layer F.Cu) (net 30))
+  (segment (start 206.12868 75.85) (end 190.9 75.85) (width 2) (layer F.Cu) (net 30))
+  (segment (start 210.87868 80.6) (end 206.12868 75.85) (width 2) (layer F.Cu) (net 30))
+  (segment (start 190.9 75.85) (end 187 75.85) (width 2) (layer F.Cu) (net 30))
+  (segment (start 213 80.6) (end 210.87868 80.6) (width 2) (layer F.Cu) (net 30))
   (segment (start 200.58 96) (end 201.5 96.92) (width 0.25) (layer F.Cu) (net 32))
   (segment (start 197.725 96) (end 200.58 96) (width 0.25) (layer F.Cu) (net 32))
@@
       )
     )
+  )
+  (zone (net 7) (net_name GND) (layer B.Cu) (hatch edge 0.508)
+    (connect_pads (clearance 0.508))
+    (min_thickness 0.254)
+    (fill yes (arc_segments 32) (thermal_gap 0.508) (thermal_bridge_width 0.508))
+    (polygon
+      (pts
+        (xy 160 148) (xy 160 70) (xy 217 70) (xy 217 148)
+      )
+    )
